File: v2..0/MosfetSchaltung_v2.sch (KiCad schematic (older format))
At the start: 31 parts, among them J3 XT60, J4 XT60, J5 XT60, Q1 IRF1404, Q2 IRF1404, Q3 IRF1404, Q4 IRF1404, SW1 LED on/off, U1 4N35, U2 4N35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

Commit message: KiCad Cicuits Files
Parts:
- removed C1: 470nF, symbol CP
- removed C2, C4: 100nF, symbol C
- removed C3: 47µF, symbol CP
- removed D1, D2: D_Sch, symbol D_Schottky
- removed D3, D4: LED, symbol LED
- removed J3, J4, J5: XT60, symbol XT60
- removed J?: Input_1, symbol Conn_01x02_Female
- removed J?: Input_2, symbol Conn_01x02_Female
- removed J?: Conn_01x03_Female, symbol Conn_01x03_Female
- removed Q1, Q2, Q3, Q4: IRF1404, TO_SOT_Packages_THT:TO-220_Vertical, symbol BUZ11
- removed R1, R2, R3, R4: 10k, symbol R
- removed R5, R6: 510, symbol R
- removed R? (x2): 330, symbol R
- removed SW1: LED on/off, symbol SW_DIP_x01
- removed U1, U2: 4N35, Housings_DIP:DIP-6_W7.62mm, symbol 4N27
- removed U3: TC4426, symbol MIC4426
- removed U4: L7810, symbol L7812
- added C1, C3: 100n, Capacitor_THT:C_Disc_D6.0mm_W4.4mm_P5.00mm, symbol Device:C
- added C2: 4,7µ, Capacitor_THT:CP_Radial_D4.0mm_P1.50mm, symbol Device:CP
- added C4: 47µ, Capacitor_THT:CP_Radial_D4.0mm_P1.50mm, symbol Device:CP
- added C5: 1000µ, Capacitor_THT:CP_Radial_D10.0mm_P5.00mm, symbol Device:CP
- added D1, D6: D_Bridge_+-AA, Diode_SMD:Diode_Bridge_Diotec_ABS, symbol Device:D_Bridge_+-AA
- added D2, D4: LED, LED_THT:LED_D3.0mm, symbol Device:LED
- added D3, D5: D_Schottky, Diode_THT:D_DO-35_SOD27_P5.08mm_Vertical_AnodeUp, symbol Device:D_Schottky
- added J1: Power Supply Input, XT60:XT60, symbol Connector_Generic:Conn_01x02
- added J2: HotBed, Connector_JST:JST_XH_B02B-XH-A_1x02_P2.50mm_Vertical, symbol Connector_Generic:Conn_01x02
- added J3: HotBed, XT60:XT60, symbol Connector_Generic:Conn_01x02
- added J4: Hotend, XT60:XT60, symbol Connector_Generic:Conn_01x02
- added J5: HotEnd, Connector_JST:JST_XH_B02B-XH-A_1x02_P2.50mm_Vertical, symbol Connector_Generic:Conn_01x02
- added J6: HotBed_direkt, Connector_JST:JST_XH_B02B-XH-A_1x02_P2.50mm_Vertical, symbol Connector_Generic:Conn_01x02
- added J7: HotEnd_direkt, Connector_JST:JST_XH_B02B-XH-A_1x02_P2.50mm_Vertical, symbol Connector_Generic:Conn_01x02
- added MH1, MH2: MountingHole, MountingHole:MountingHole_3.2mm_M3, symbol Mechanical:MountingHole
- added Q1, Q2, Q3: N-Channel_Mosfet, Package_TO_SOT_THT:TO-220-3_Vertical, symbol Transistor_FET:IRLZ44N
- added R1, R6: 512, Resistor_THT:R_Axial_DIN0207_L6.3mm_D2.5mm_P5.08mm_Vertical, symbol Device:R
- added R10, R9: 0, Resistor_SMD:R_0402_1005Metric, symbol Device:R
- added R2, R3, R7, R8: 10k, Resistor_THT:R_Axial_DIN0207_L6.3mm_D2.5mm_P5.08mm_Vertical, symbol Device:R
- added R4, R5: 2,2k, Resistor_THT:R_Axial_DIN0207_L6.3mm_D2.5mm_P5.08mm_Vertical, symbol Device:R
- added SW1: Led On/Off, Connector_PinSocket_2.54mm:PinSocket_1x03_P2.54mm_Vertical, symbol Switch:SW_Push_SPDT
- added TP1, TP2, TP3: TestPoint, TestPoint:TestPoint_THTPad_3.0x3.0mm_Drill1.5mm, symbol Connector:TestPoint
- added U1, U3: 4N35, Package_DIP:DIP-6_W7.62mm, symbol Isolator:4N35
- added U2: TC4426CPA, Package_DIP:DIP-8_W7.62mm, symbol TC4426CPA:TC4426CPA
- added U4: L7810, Package_TO_SOT_THT:TO-220-3_Vertical, symbol Regulator_Linear:L7812
Connections:
- net labels added: +10V
- net labels removed: +12V
- wire segments 87 -> 112
Other:
- note removed: "Hotbed Connector"
- note removed: "Hotend Connector"
- note removed: "Power Supply Input"
